Commit message: Adding the xacro files

File: urdf/base.xacro (robot description, xacro)
@@ -1,9 +1,7 @@
 <?xml version="1.0" ?>
 <robot name="cratebot" xmlns:xacro="http://www.ros.org/wiki/xacro">
-    <!--
     <xacro:include filename="$(find cratebot_description)/urdf/materials.xacro" />
     <xacro:include filename="$(find cratebot_description)/urdf/transmittions.xacro" />
     <xacro:include filename="$(find cratebot_description)/urdf/gazebo.xacro" />
-    -->
     <!--
       An empty base link for the following reasons:
@@ -52,5 +50,5 @@
                 <box size="0.35, 0.2, 0.06" />
             </geometry>
-            <!-- <material name="silver"/> -->
+            <material name="silver"/>
         </visual>
         <collision>
@@ -76,10 +74,23 @@
                 <cylinder length="0.01" radius="0.05" />
             </geometry>
-            <!-- <material name="black"/> -->
-        </visual>
-        <collision>
-            <origin rpy="0 0 0" xyz="0 0 0"/>
-            <geometry>
-                <cylinder length="0.01" radius="0.05" />
+            <material name="blue"/>
+        </visual>
+        <collision>
+            <origin rpy="0 0 0" xyz="0 0 0"/>
+            <geometry>
+                <cylinder length="0.01" radius="0.05" />
+            </geometry>
+        </collision>
+        <visual>
+            <origin rpy="0 0 0" xyz="0 -0.04 -0.035"/>
+            <geometry>
+                <box size="0.04, 0.01, 0.06" />
+            </geometry>
+            <material name="blue"/>
+        </visual>
+        <collision>
+            <origin rpy="0 0 0" xyz="0 -0.04 -0.035"/>
+            <geometry>
+                <box size="0.04, 0.01, 0.06" />
             </geometry>
         </collision>
@@ -97,5 +108,5 @@
                 <cylinder length="0.05" radius="0.04" />
             </geometry>
-            <!-- <material name="black"/> -->
+            <material name="black"/>
         </visual>
         <collision>
@@ -121,10 +132,23 @@
                 <cylinder length="0.01" radius="0.05" />
             </geometry>
-            <!-- <material name="black"/> -->
-        </visual>
-        <collision>
-            <origin rpy="0 0 0" xyz="0 0 0"/>
-            <geometry>
-                <cylinder length="0.01" radius="0.05" />
+            <material name="blue"/>
+        </visual>
+        <collision>
+            <origin rpy="0 0 0" xyz="0 0 0"/>
+            <geometry>
+                <cylinder length="0.01" radius="0.05" />
+            </geometry>
+        </collision>
+        <visual>
+            <origin rpy="0 0 0" xyz="0 0.04 -0.035"/>
+            <geometry>
+                <box size="0.04, 0.01, 0.06" />
+            </geometry>
+            <material name="blue"/>
+        </visual>
+        <collision>
+            <origin rpy="0 0 0" xyz="0 0.04 -0.035"/>
+            <geometry>
+                <box size="0.04, 0.01, 0.06" />
             </geometry>
         </collision>
@@ -142,5 +166,5 @@
                 <cylinder length="0.05" radius="0.04" />
             </geometry>
-            <!-- <material name="black"/> -->
+            <material name="black"/>
         </visual>
         <collision>
@@ -166,10 +190,23 @@
                 <cylinder length="0.01" radius="0.05" />
             </geometry>
-            <!-- <material name="black"/> -->
-        </visual>
-        <collision>
-            <origin rpy="0 0 0" xyz="0 0 0"/>
-            <geometry>
-                <cylinder length="0.01" radius="0.05" />
+            <material name="blue"/>
+        </visual>
+        <collision>
+            <origin rpy="0 0 0" xyz="0 0 0"/>
+            <geometry>
+                <cylinder length="0.01" radius="0.05" />
+            </geometry>
+        </collision>
+        <visual>
+            <origin rpy="0 0 0" xyz="0 -0.04 -0.035"/>
+            <geometry>
+                <box size="0.04, 0.01, 0.06" />
+            </geometry>
+            <material name="blue"/>
+        </visual>
+        <collision>
+            <origin rpy="0 0 0" xyz="0 -0.04 -0.035"/>
+            <geometry>
+                <box size="0.04, 0.01, 0.06" />
             </geometry>
         </collision>
@@ -187,5 +224,5 @@
                 <cylinder length="0.05" radius="0.04" />
             </geometry>
-            <!-- <material name="black"/> -->
+            <material name="black"/>
         </visual>
         <collision>
@@ -211,10 +248,23 @@
                 <cylinder length="0.01" radius="0.05" />
             </geometry>
-            <!-- <material name="black"/> -->
-        </visual>
-        <collision>
-            <origin rpy="0 0 0" xyz="0 0 0"/>
-            <geometry>
-                <cylinder length="0.01" radius="0.05" />
+            <material name="blue"/>
+        </visual>
+        <collision>
+            <origin rpy="0 0 0" xyz="0 0 0"/>
+            <geometry>
+                <cylinder length="0.01" radius="0.05" />
+            </geometry>
+        </collision>
+        <visual>
+            <origin rpy="0 0 0" xyz="0 0.04 -0.035"/>
+            <geometry>
+                <box size="0.04, 0.01, 0.06" />
+            </geometry>
+            <material name="blue"/>
+        </visual>
+        <collision>
+            <origin rpy="0 0 0" xyz="0 0.04 -0.035"/>
+            <geometry>
+                <box size="0.04, 0.01, 0.06" />
             </geometry>
         </collision>
@@ -232,5 +282,5 @@
                 <cylinder length="0.05" radius="0.04" />
             </geometry>
-            <!-- <material name="black"/> -->
+            <material name="black"/>
         </visual>
         <collision>

Commit message: Don't put comma's in the xacro files

File: urdf/base.xacro (robot description, xacro)
@@ -48,5 +48,5 @@
             <origin rpy="0 0 0" xyz="0 0 0.07"/>
             <geometry>
-                <box size="0.35, 0.2, 0.06" />
+                <box size="0.35 0.2 0.06" />
             </geometry>
             <material name="silver"/>
@@ -55,5 +55,5 @@
             <origin rpy="0 0 0" xyz="0 0 0.07"/>
             <geometry>
-                <box size="0.35, 0.2, 0.06" />
+                <box size="0.35 0.2 0.06" />
             </geometry>
         </collision>
@@ -85,12 +85,12 @@
             <origin rpy="0 0 0" xyz="0 -0.04 -0.035"/>
             <geometry>
-                <box size="0.04, 0.01, 0.06" />
-            </geometry>
-            <material name="blue"/>
-        </visual>
-        <collision>
-            <origin rpy="0 0 0" xyz="0 -0.04 -0.035"/>
-            <geometry>
-                <box size="0.04, 0.01, 0.06" />
+                <box size="0.04 0.01 0.06" />
+            </geometry>
+            <material name="blue"/>
+        </visual>
+        <collision>
+            <origin rpy="0 0 0" xyz="0 -0.04 -0.035"/>
+            <geometry>
+                <box size="0.04 0.01 0.06" />
             </geometry>
         </collision>
@@ -143,12 +143,12 @@
             <origin rpy="0 0 0" xyz="0 0.04 -0.035"/>
             <geometry>
-                <box size="0.04, 0.01, 0.06" />
-            </geometry>
-            <material name="blue"/>
-        </visual>
-        <collision>
-            <origin rpy="0 0 0" xyz="0 0.04 -0.035"/>
-            <geometry>
-                <box size="0.04, 0.01, 0.06" />
+                <box size="0.04 0.01 0.06" />
+            </geometry>
+            <material name="blue"/>
+        </visual>
+        <collision>
+            <origin rpy="0 0 0" xyz="0 0.04 -0.035"/>
+            <geometry>
+                <box size="0.04 0.01 0.06" />
             </geometry>
         </collision>
@@ -201,12 +201,12 @@
             <origin rpy="0 0 0" xyz="0 -0.04 -0.035"/>
             <geometry>
-                <box size="0.04, 0.01, 0.06" />
-            </geometry>
-            <material name="blue"/>
-        </visual>
-        <collision>
-            <origin rpy="0 0 0" xyz="0 -0.04 -0.035"/>
-            <geometry>
-                <box size="0.04, 0.01, 0.06" />
+                <box size="0.04 0.01 0.06" />
+            </geometry>
+            <material name="blue"/>
+        </visual>
+        <collision>
+            <origin rpy="0 0 0" xyz="0 -0.04 -0.035"/>
+            <geometry>
+                <box size="0.04 0.01 0.06" />
             </geometry>
         </collision>
@@ -259,12 +259,12 @@
             <origin rpy="0 0 0" xyz="0 0.04 -0.035"/>
             <geometry>
-                <box size="0.04, 0.01, 0.06" />
-            </geometry>
-            <material name="blue"/>
-        </visual>
-        <collision>
-            <origin rpy="0 0 0" xyz="0 0.04 -0.035"/>
-            <geometry>
-                <box size="0.04, 0.01, 0.06" />
+                <box size="0.04 0.01 0.06" />
+            </geometry>
+            <material name="blue"/>
+        </visual>
+        <collision>
+            <origin rpy="0 0 0" xyz="0 0.04 -0.035"/>
+            <geometry>
+                <box size="0.04 0.01 0.06" />
             </geometry>
         </collision>

Commit message: Add inertia

File: urdf/base.xacro (robot description, xacro)
@@ -9,6 +9,6 @@
         its inertia defined. So the fix is to define a 'dummy' base link.
     -->
-    <link name="base_link">
-    </link>
+    <!-- <link name="base_link">
+    </link> -->
     <!--
         A box that pretends to be the ground. Used for testing that the scuttle model has been assembled correctly.
@@ -30,4 +30,5 @@
         as the child frame.
     -->
+    <!--
     <joint name="chassis_joint" type="fixed">
         <origin rpy="0 0 0" xyz="0.0 0 0.0"/>
@@ -35,4 +36,5 @@
         <child link="chassis_link"/>
     </joint>
+    -->
     <!--
       The coordinate framework has the X-asis in the direction of forward motion, with the y-axis pointing
@@ -40,11 +42,9 @@
     -->
     <link name="chassis_link">
-        <!--
-        <inertial>
-            <origin rpy="0 0 0" xyz="2.12433370053547e-05 -0.07877992189559235 0.07392564365565002"/>
-            <mass value="3.288323846275119"/>
-            <inertia ixx="0.038876" ixy="1.3e-05" ixz="1e-06" iyy="0.047513" iyz="0.000486" izz="0.084083"/>
-        </inertial>
-        -->
+        <inertial>
+            <origin rpy="0 0 0" xyz="0 0 0.07"/>
+            <mass value="1.0"/>
+            <inertia ixx="0.00363" ixy="0" ixz="0" iyy="0.0105" iyz="0" izz="0.0135"/>
+        </inertial>
         <visual>
             <origin rpy="0 0 0" xyz="0 0 0.07"/>
@@ -71,4 +71,9 @@
     </joint>
     <link name="left_front_wheel_swivel_link">
+        <inertial>
+            <origin rpy="0 0 0" xyz="0 0 0"/>
+            <mass value="0.2"/>
+            <inertia ixx="0.001" ixy="0" ixz="0" iyy="0.01" iyz="0" izz="0.01"/>
+        </inertial>
         <visual>
             <origin rpy="0 0 0" xyz="0 0 0"/>
@@ -105,4 +110,9 @@
     </joint>
     <link name="left_front_wheel_link">
+        <inertial>
+            <origin rpy="0 0 0" xyz="0 0 0"/>
+            <mass value="0.2"/>
+            <inertia ixx="0.001" ixy="0" ixz="0" iyy="0.01" iyz="0" izz="0.01"/>
+        </inertial>
         <visual>
             <origin rpy="0 0 0" xyz="0 0 0"/>
@@ -129,4 +139,9 @@
     </joint>
     <link name="right_front_wheel_swivel_link">
+        <inertial>
+            <origin rpy="0 0 0" xyz="0 0 0"/>
+            <mass value="0.2"/>
+            <inertia ixx="0.001" ixy="0" ixz="0" iyy="0.01" iyz="0" izz="0.01"/>
+        </inertial>
         <visual>
             <origin rpy="0 0 0" xyz="0 0 0"/>
@@ -163,4 +178,9 @@
     </joint>
     <link name="right_front_wheel_link">
+        <inertial>
+            <origin rpy="0 0 0" xyz="0 0 0"/>
+            <mass value="0.2"/>
+            <inertia ixx="0.001" ixy="0" ixz="0" iyy="0.01" iyz="0" izz="0.01"/>
+        </inertial>
         <visual>
             <origin rpy="0 0 0" xyz="0 0 0"/>
@@ -187,4 +207,9 @@
     </joint>
     <link name="left_rear_wheel_swivel_link">
+        <inertial>
+            <origin rpy="0 0 0" xyz="0 0 0"/>
+            <mass value="0.2"/>
+            <inertia ixx="0.001" ixy="0" ixz="0" iyy="0.01" iyz="0" izz="0.01"/>
+        </inertial>
         <visual>
             <origin rpy="0 0 0" xyz="0 0 0"/>
@@ -221,4 +246,9 @@
     </joint>
     <link name="left_rear_wheel_link">
+        <inertial>
+            <origin rpy="0 0 0" xyz="0 0 0"/>
+            <mass value="0.2"/>
+            <inertia ixx="0.001" ixy="0" ixz="0" iyy="0.01" iyz="0" izz="0.01"/>
+        </inertial>
         <visual>
             <origin rpy="0 0 0" xyz="0 0 0"/>
@@ -245,4 +275,9 @@
     </joint>
     <link name="right_rear_wheel_swivel_link">
+        <inertial>
+            <origin rpy="0 0 0" xyz="0 0 0"/>
+            <mass value="0.2"/>
+            <inertia ixx="0.001" ixy="0" ixz="0" iyy="0.01" iyz="0" izz="0.01"/>
+        </inertial>
         <visual>
             <origin rpy="0 0 0" xyz="0 0 0"/>
@@ -279,4 +314,9 @@
     </joint>
     <link name="right_rear_wheel_link">
+        <inertial>
+            <origin rpy="0 0 0" xyz="0 0 0"/>
+            <mass value="0.2"/>
+            <inertia ixx="0.001" ixy="0" ixz="0" iyy="0.01" iyz="0" izz="0.01"/>
+        </inertial>
         <visual>
             <origin rpy="0 0 0" xyz="0 0 0"/>
