Commit message: Introducing the use_fake_hardware switch so that we can run without gazebo

File: urdf/base.xacro (robot description, xacro)
@@ -1,12 +1,11 @@
 <?xml version="1.0" ?>
 <robot name="cratebot" xmlns:xacro="http://www.ros.org/wiki/xacro">
-    <xacro:include filename="$(find cratebot_description)/urdf/materials.xacro" />
-    <xacro:include filename="$(find cratebot_description)/urdf/macros.xacro" />
-    <xacro:include filename="$(find cratebot_description)/urdf/gazebo.xacro" />
     <!-- CONSTANTS -->
     <!-- Math -->
     <xacro:property name="PI" value="3.1415926535897931"/>
-    <!-- -->
+    <!-- ARGUMENTS -->
     <xacro:arg name="is_simulation" default="true" />
+    <xacro:arg name="use_fake_hardware" default="true" />
+    <xacro:arg name="fake_sensor_commands" default="false" />
     <!-- Chassis dimensions -->
     <xacro:property name="chassis_mass" value="1.0" /> <!-- arbitrary value for base mass -->
@@ -28,5 +27,10 @@
     <xacro:property name="left_y_reflect" value="-1" />
     <xacro:property name="right_y_reflect" value="1" />
-    <!-- MACROS -->
+    <!-- INCLUDES -->
+    <xacro:include filename="$(find cratebot_description)/urdf/materials.xacro" />
+    <xacro:include filename="$(find cratebot_description)/urdf/macros.xacro" />
+    <xacro:if value="${is_simulation}">
+    <xacro:include filename="$(find cratebot_description)/urdf/gazebo.xacro" />
+    </xacro:if>
     <!-- MODEL -->
     <!--
@@ -126,5 +130,6 @@
         x_reflect="${front_x_reflect}"
         y_reflect="${left_y_reflect}"
-        is_simulation="$(arg is_simulation)" />
+        is_simulation="$(arg is_simulation)"
+        use_fake_hardware="$(arg use_fake_hardware)" />
     <!--
         Right front wheel assembly
@@ -144,5 +149,6 @@
         x_reflect="${front_x_reflect}"
         y_reflect="${right_y_reflect}"
-        is_simulation="$(arg is_simulation)" />
+        is_simulation="$(arg is_simulation)"
+        use_fake_hardware="$(arg use_fake_hardware)" />
     <!--
         Left rear wheel assembly
@@ -162,5 +168,6 @@
         x_reflect="${rear_x_reflect}"
         y_reflect="${left_y_reflect}"
-        is_simulation="$(arg is_simulation)" />
+        is_simulation="$(arg is_simulation)"
+        use_fake_hardware="$(arg use_fake_hardware)" />
     <!--
         Right rear wheel assembly
@@ -180,4 +187,5 @@
         x_reflect="${rear_x_reflect}"
         y_reflect="${right_y_reflect}"
-        is_simulation="$(arg is_simulation)" />
+        is_simulation="$(arg is_simulation)"
+        use_fake_hardware="$(arg use_fake_hardware)" />
 </robot>

File: urdf/macros.xacro (robot description, xacro)
@@ -120,5 +120,5 @@
         - y_reflect: Direction multiplier for Y offsets. Either 1 or -1
     -->
-    <xacro:macro name="drive_module_assembly" params="name chassis_length chassis_width chassis_height wheel_mass wheel_radius wheel_width steering_mass steering_radius steering_thickness offset x_reflect y_reflect is_simulation">
+    <xacro:macro name="drive_module_assembly" params="name chassis_length chassis_width chassis_height wheel_mass wheel_radius wheel_width steering_mass steering_radius steering_thickness offset x_reflect y_reflect is_simulation use_fake_hardware">
         <xacro:steering_assembly
             name="${name}"
@@ -141,8 +141,9 @@
         <xacro:steering_module_controller
             name="${name}"
-            is_simulation="${is_simulation}" />
+            is_simulation="${is_simulation}"
+            use_fake_hardware="${use_fake_hardware}" />
     </xacro:macro>
     <!-- CONTROLLERS -->
-    <xacro:macro name="steering_module_controller" params="name is_simulation:=^|true">
+    <xacro:macro name="steering_module_controller" params="name is_simulation:=^|true use_fake_hardware:=^|false">
         <ros2_control name="control_steering_${name}" type="system">
             <hardware>
@@ -152,4 +153,10 @@
                 </xacro:if>
                 <xacro:unless value="${is_simulation}">
+                    <xacro:if value="${use_fake_hardware}">
+                        <plugin>mock_components/GenericSystem</plugin>
+                    </xacro:if>
+                    <xacro:unless value="${use_fake_hardware}">
+                        <!-- USE REAL HARDWARE HERE -->
+                    </xacro:unless>
                 </xacro:unless>
             </hardware>

Commit message: Merging the ros control sections for each steering module into one section.

File: urdf/base.xacro (robot description, xacro)
@@ -8,4 +8,5 @@
     <xacro:arg name="use_fake_hardware" default="true" />
     <xacro:arg name="fake_sensor_commands" default="false" />
+    <xacro:arg name="chassis_version" default="v1" />
     <!-- Chassis dimensions -->
     <xacro:property name="chassis_mass" value="1.0" /> <!-- arbitrary value for base mass -->
@@ -129,7 +130,5 @@
         offset="${wheel_offset}"
         x_reflect="${front_x_reflect}"
-        y_reflect="${left_y_reflect}"
-        is_simulation="$(arg is_simulation)"
-        use_fake_hardware="$(arg use_fake_hardware)" />
+        y_reflect="${left_y_reflect}" />
     <!--
         Right front wheel assembly
@@ -148,7 +147,5 @@
         offset="${wheel_offset}"
         x_reflect="${front_x_reflect}"
-        y_reflect="${right_y_reflect}"
-        is_simulation="$(arg is_simulation)"
-        use_fake_hardware="$(arg use_fake_hardware)" />
+        y_reflect="${right_y_reflect}" />
     <!--
         Left rear wheel assembly
@@ -167,7 +164,5 @@
         offset="${wheel_offset}"
         x_reflect="${rear_x_reflect}"
-        y_reflect="${left_y_reflect}"
-        is_simulation="$(arg is_simulation)"
-        use_fake_hardware="$(arg use_fake_hardware)" />
+        y_reflect="${left_y_reflect}" />
     <!--
         Right rear wheel assembly
@@ -186,6 +181,28 @@
         offset="${wheel_offset}"
         x_reflect="${rear_x_reflect}"
-        y_reflect="${right_y_reflect}"
-        is_simulation="$(arg is_simulation)"
-        use_fake_hardware="$(arg use_fake_hardware)" />
+        y_reflect="${right_y_reflect}" />
+    <ros2_control name="CratebotJointControl" type="system">
+        <xacro:if value="${is_simulation}">
+            <hardware>
+                <plugin>ign_ros2_control/IgnitionSystem</plugin>
+                <param name="example_param_read_for_sec">0.43</param>
+            </hardware>
+        </xacro:if>
+        <xacro:unless value="${is_simulation}">
+            <xacro:if value="${use_fake_hardware}">
+                <hardware>
+                    <plugin>mock_components/GenericSystem</plugin>
+                </hardware>
+            </xacro:if>
+            <xacro:unless value="${use_fake_hardware}">
+                <!-- USE REAL HARDWARE HERE -->
+                <hardware>
+                </hardware>
+            </xacro:unless>
+        </xacro:unless>
+        <xacro:steering_module_controller name="left_front" />
+        <xacro:steering_module_controller name="right_front" />
+        <xacro:steering_module_controller name="left_rear" />
+        <xacro:steering_module_controller name="right_rear" />
+    </ros2_control>
 </robot>

File: urdf/macros.xacro (robot description, xacro)
@@ -120,5 +120,5 @@
         - y_reflect: Direction multiplier for Y offsets. Either 1 or -1
     -->
-    <xacro:macro name="drive_module_assembly" params="name chassis_length chassis_width chassis_height wheel_mass wheel_radius wheel_width steering_mass steering_radius steering_thickness offset x_reflect y_reflect is_simulation use_fake_hardware">
+    <xacro:macro name="drive_module_assembly" params="name chassis_length chassis_width chassis_height wheel_mass wheel_radius wheel_width steering_mass steering_radius steering_thickness offset x_reflect y_reflect">
         <xacro:steering_assembly
             name="${name}"
@@ -139,45 +139,25 @@
             width="${wheel_width}"
             offset="${offset}"/>
-        <xacro:steering_module_controller
-            name="${name}"
-            is_simulation="${is_simulation}"
-            use_fake_hardware="${use_fake_hardware}" />
     </xacro:macro>
     <!-- CONTROLLERS -->
-    <xacro:macro name="steering_module_controller" params="name is_simulation:=^|true use_fake_hardware:=^|false">
-        <ros2_control name="control_steering_${name}" type="system">
-            <hardware>
-                <xacro:if value="${is_simulation}">
-                    <plugin>ign_ros2_control/IgnitionSystem</plugin>
-                    <param name="example_param_read_for_sec">0.43</param>
-                </xacro:if>
-                <xacro:unless value="${is_simulation}">
-                    <xacro:if value="${use_fake_hardware}">
-                        <plugin>mock_components/GenericSystem</plugin>
-                    </xacro:if>
-                    <xacro:unless value="${use_fake_hardware}">
-                        <!-- USE REAL HARDWARE HERE -->
-                    </xacro:unless>
-                </xacro:unless>
-            </hardware>
-            <joint name="joint_chassis_to_steering_${name}">
-                <command_interface name="position">
-                    <param name="min">-1</param>
-                    <param name="max">1</param>
-                </command_interface>
-                <state_interface name="position"/>
-                <state_interface name="velocity"/>
-                <state_interface name="effort"/>
-            </joint>
-            <joint name="joint_steering_to_wheel_${name}">
-                <command_interface name="velocity">
-                    <param name="min">-1</param>
-                    <param name="max">1</param>
-                </command_interface>
-                <state_interface name="position"/>
-                <state_interface name="velocity"/>
-                <state_interface name="effort"/>
-            </joint>
-        </ros2_control>
+    <xacro:macro name="steering_module_controller" params="name">
+        <joint name="joint_chassis_to_steering_${name}">
+            <command_interface name="position">
+                <param name="min">-1</param>
+                <param name="max">1</param>
+            </command_interface>
+            <state_interface name="position"/>
+            <state_interface name="velocity"/>
+            <state_interface name="effort"/>
+        </joint>
+        <joint name="joint_steering_to_wheel_${name}">
+            <command_interface name="velocity">
+                <param name="min">-1</param>
+                <param name="max">1</param>
+            </command_interface>
+            <state_interface name="position"/>
+            <state_interface name="velocity"/>
+            <state_interface name="effort"/>
+        </joint>
     </xacro:macro>
 </robot>

Commit message: Swap the base_footprint and base_link joints

File: urdf/base.xacro (robot description, xacro)
@@ -36,10 +36,10 @@
     <!-- MODEL -->
     <!--
+      An empty base footprint that describes the origin of the robot on the ground
+    -->
+    <link name="base_footprint">
+    </link>
+    <!--
       An empty base link that describes the origin of the robot at the c.o.g of the chassis
-    -->
-    <link name="base_link">
-    </link>
-    <!--
-      An empty base footprint that describes the origin of the robot on the ground
     -->
     <!--
@@ -49,9 +49,9 @@
     -->
     <joint name="joint_base_to_footprint" type="fixed">
-        <origin rpy="0 0 0" xyz="0 0 -${wheel_radius + 0.5 * chassis_height}"/>
-        <parent link="base_link"/>
-        <child link="base_footprint"/>
+        <origin rpy="0 0 0" xyz="0 0 ${wheel_radius + 0.5 * chassis_height}"/>
+        <parent link="base_footprint"/>
+        <child link="base_link"/>
     </joint>
-    <link name="base_footprint">
+    <link name="base_link">
     </link>
     <!--

Commit message: Fix issues in the URDF

File: urdf/base.xacro (robot description, xacro)
@@ -26,6 +26,6 @@
     <xacro:property name="front_x_reflect" value="1" />
     <xacro:property name="rear_x_reflect" value="-1" />
-    <xacro:property name="left_y_reflect" value="-1" />
-    <xacro:property name="right_y_reflect" value="1" />
+    <xacro:property name="left_y_reflect" value="1" />
+    <xacro:property name="right_y_reflect" value="-1" />
     <!-- INCLUDES -->
     <xacro:include filename="$(find cratebot_description)/urdf/materials.xacro" />

File: urdf/macros.xacro (robot description, xacro)
@@ -138,5 +138,5 @@
             radius="${wheel_radius}"
             width="${wheel_width}"
-            offset="${offset}"/>
+            offset="${offset + 0.5 * steering_thickness}"/>
     </xacro:macro>
     <!-- CONTROLLERS -->

Commit message: Adding a lidar and an IMU to the robot

File: urdf/base.xacro (robot description, xacro)
@@ -105,5 +105,5 @@
                 <box size="${chassis_length} ${chassis_width} ${chassis_height}" />
             </geometry>
-            <material name="silver"/>
+            <material name="orange"/>
         </visual>
         <collision>
@@ -205,3 +205,16 @@
         <xacro:steering_module_controller name="right_front" />
     </ros2_control>
+    <!-- Sensors -->
+    <!-- IMU -->
+    <xacro:sensor_imu name="imu_center" parent_link="chassis_link">
+        <origin rpy="0 0 0" xyz="0.0 0.0 0.0"/>
+    </xacro:sensor_imu>
+    <!-- LIDAR -->
+    <xacro:sensor_lidar name="rplidar_front" parent_link="chassis_link">
+        <origin rpy="0 0 0" xyz="0.0 0.0 0.0"/>
+    </xacro:sensor_lidar>
+    <!-- Bump -->
+    <!-- Sonar -->
+    <!-- IR -->
+    <!-- Cliff sensors -->
 </robot>

File: urdf/gazebo.xacro (robot description, xacro)
@@ -20,4 +20,90 @@
         </gazebo>
     </xacro:macro>
+    <xacro:macro name="gazebo_sensor_rplidar" params="name" >
+        <gazebo reference="link_sensor_lidar_${name}">
+            <sensor name="${name}" type="gpu_lidar">
+                <update_rate>62.0</update_rate>
+                <visualize>1</visualize>
+                <always_on>true</always_on>
+                <lidar>
+                <scan>
+                    <horizontal>
+                        <samples>640</samples>
+                        <resolution>1.0</resolution>
+                        <min_angle>${-pi}</min_angle>
+                        <max_angle>${pi}</max_angle>
+                    </horizontal>
+                    <vertical>
+                        <samples>1</samples>
+                        <resolution>1</resolution>
+                        <min_angle>0</min_angle>
+                        <max_angle>0</max_angle>
+                    </vertical>
+                </scan>
+                <range>
+                    <min>0.164</min>
+                    <max>12.0</max>
+                    <resolution>0.01</resolution>
+                </range>
+                </lidar>
+            </sensor>
+        </gazebo>
+        <gazebo reference="joint_body_to_sensor_lidar_${name}">
+            <preserveFixedJoint>true</preserveFixedJoint>
+        </gazebo>
+    </xacro:macro>
+    <xacro:macro name="gazebo_sensor_imu" params="name update_rate:=62" >
+        <gazebo reference="link_sensor_imu_${name}">
+            <sensor name="${name}" type="imu">
+                <always_on>true</always_on>
+                <update_rate>${update_rate}</update_rate>
+                <imu>
+                    <angular_velocity>
+                    <x>
+                        <noise type="gaussian">
+                        <mean>0.0</mean>
+                        <stddev>0.0</stddev>
+                        </noise>
+                    </x>
+                    <y>
+                        <noise type="gaussian">
+                        <mean>0.0</mean>
+                        <stddev>0.0</stddev>
+                        </noise>
+                    </y>
+                    <z>
+                        <noise type="gaussian">
+                        <mean>0.0</mean>
+                        <stddev>0.0</stddev>
+                        </noise>
+                    </z>
+                    </angular_velocity>
+                    <linear_acceleration>
+                    <x>
+                        <noise type="gaussian">
+                        <mean>0.0</mean>
+                        <stddev>0.0</stddev>
+                        </noise>
+                    </x>
+                    <y>
+                        <noise type="gaussian">
+                        <mean>0.0</mean>
+                        <stddev>0.0</stddev>
+                        </noise>
+                    </y>
+                    <z>
+                        <noise type="gaussian">
+                        <mean>0.0</mean>
+                        <stddev>0.0</stddev>
+                        </noise>
+                    </z>
+                    </linear_acceleration>
+                </imu>
+            </sensor>
+        </gazebo>
+        <gazebo reference="joint_body_to_sensor_imu_${name}">
+            <preserveFixedJoint>true</preserveFixedJoint>
+        </gazebo>
+    </xacro:macro>
     <!--
         GAZEBO
@@ -27,4 +113,6 @@
     <xacro:gazebo_reference_link_wheel name="right_rear" />
     <xacro:gazebo_reference_link_wheel name="right_front" />
+    <xacro:gazebo_sensor_rplidar name="rplidar_front" />
+    <xacro:gazebo_sensor_imu name="imu_center" />
     <gazebo>
         <plugin

File: urdf/macros.xacro (robot description, xacro)
@@ -161,3 +161,87 @@
         </joint>
     </xacro:macro>
+    <!-- SENSORS -->
+    <!-- Lidar sensor -->
+    <xacro:macro name="sensor_lidar" params="name parent_link *origin">
+        <xacro:property name="mass"     value="0.17"/>
+        <xacro:property name="length_x" value="0.071" />
+        <xacro:property name="length_y" value="0.10" />
+        <xacro:property name="length_z" value="0.06" />
+        <xacro:property name="collision_x_offset" value="0" />
+        <xacro:property name="collision_y_offset" value="0.013" />
+        <xacro:property name="collision_z_offset" value="-0.019" />
+        <joint name="joint_body_to_sensor_lidar_${name}" type="fixed">
+            <parent link="${parent_link}"/>
+            <child link="link_sensor_lidar_${name}"/>
+            <xacro:insert_block name="origin"/>
+        </joint>
+        <link name="link_sensor_lidar_${name}">
+            <visual>
+                <origin xyz="${collision_x_offset} ${collision_y_offset} ${collision_z_offset}"/>
+                <geometry>
+                    <box size="${length_x} ${length_y} ${length_z}"/>
+                </geometry>
+            </visual>
+            <collision>
+                <origin xyz="${collision_x_offset} ${collision_y_offset} ${collision_z_offset}"/>
+                <geometry>
+                    <box size="${length_x} ${length_y} ${length_z}"/>
+                </geometry>
+            </collision>
+            <inertial>
+                <mass value="${mass}" />
+                <xacro:insert_block name="origin"/>
+                <inertia
+                    ixx="${(1/12) * ${mass} * (${length_y}*${length_y} + ${length_z}*${length_z})}"
+                    ixy="0.0"
+                    ixz="0.0"
+                    iyy="${(1/12) * ${mass} * (${length_x}*${length_x} + ${length_z}*${length_z})}"
+                    iyz="0.0"
+                    izz="${(1/12) * ${mass} * (${length_x}*${length_x} + ${length_y}*${length_y})}" />
+            </inertial>
+        </link>
+    </xacro:macro>
+    <!-- IMU sensor -->
+    <xacro:macro name="sensor_imu" params="name parent_link *origin">
+        <xacro:property name="mass"     value="0.01"/>
+        <xacro:property name="length_x" value="0.01" />
+        <xacro:property name="length_y" value="0.01" />
+        <xacro:property name="length_z" value="0.01" />
+        <xacro:property name="collision_x_offset" value="0.005" />
+        <xacro:property name="collision_y_offset" value="0.005" />
+        <xacro:property name="collision_z_offset" value="0.005" />
+        <joint name="joint_body_to_sensor_${name}" type="fixed">
+            <xacro:insert_block name="origin"/>
+            <parent link="${parent_link}"/>
+            <child link="link_sensor_imu_${name}"/>
+        </joint>
+        <link name="link_sensor_imu_${name}">
+            <visual>
+                <origin xyz="${collision_x_offset} ${collision_y_offset} ${collision_z_offset}"/>
+                <geometry>
+                    <box size="${length_x} ${length_y} ${length_z}"/>
+                </geometry>
+            </visual>
+            <collision>
+                <origin xyz="${collision_x_offset} ${collision_y_offset} ${collision_z_offset}"/>
+                <geometry>
+                    <box size="${length_x} ${length_y} ${length_z}"/>
+                </geometry>
+            </collision>
+            <inertial>
+                <mass value="${mass}" />
+                <xacro:insert_block name="origin"/>
+                <inertia
+                    ixx="${(1/12) * ${mass} * (${length_y}*${length_y} + ${length_z}*${length_z})}"
+                    ixy="0.0"
+                    ixz="0.0"
+                    iyy="${(1/12) * ${mass} * (${length_x}*${length_x} + ${length_z}*${length_z})}"
+                    iyz="0.0"
+                    izz="${(1/12) * ${mass} * (${length_x}*${length_x} + ${length_y}*${length_y})}" />
+            </inertial>
+        </link>
+    </xacro:macro>
+    <!-- Bump sensor -->
+    <!-- Sonar sensor -->
+    <!-- IR sensor -->
 </robot>

File: urdf/materials.xacro (robot description, xacro)
@@ -13,3 +13,6 @@
         <color rgba="0.000 0.000 0.700 1.000"/>
     </material>
+    <material name="orange">
+        <color rgba="1.000 0.624 0.000 1.000"/>
+    </material>
 </robot>
