Commit message: Move the lidar and the IMU

File: urdf/base.xacro (robot description, xacro)
@@ -212,5 +212,5 @@
     <!-- LIDAR -->
     <xacro:sensor_lidar name="rplidar_front" parent_link="chassis_link">
-        <origin rpy="0 0 0" xyz="0.0 0.0 0.0"/>
+        <origin rpy="0 0 0" xyz="0 0 ${0.5 * chassis_height}"/>
     </xacro:sensor_lidar>
     <!-- Bump -->

File: urdf/gazebo.xacro (robot description, xacro)
@@ -20,37 +20,5 @@
         </gazebo>
     </xacro:macro>
-    <xacro:macro name="gazebo_sensor_rplidar" params="name" >
-        <gazebo reference="link_sensor_lidar_${name}">
-            <sensor name="${name}" type="gpu_lidar">
-                <update_rate>62.0</update_rate>
-                <visualize>1</visualize>
-                <always_on>true</always_on>
-                <lidar>
-                <scan>
-                    <horizontal>
-                        <samples>640</samples>
-                        <resolution>1.0</resolution>
-                        <min_angle>${-pi}</min_angle>
-                        <max_angle>${pi}</max_angle>
-                    </horizontal>
-                    <vertical>
-                        <samples>1</samples>
-                        <resolution>1</resolution>
-                        <min_angle>0</min_angle>
-                        <max_angle>0</max_angle>
-                    </vertical>
-                </scan>
-                <range>
-                    <min>0.164</min>
-                    <max>12.0</max>
-                    <resolution>0.01</resolution>
-                </range>
-                </lidar>
-            </sensor>
-        </gazebo>
-        <gazebo reference="joint_body_to_sensor_lidar_${name}">
-            <preserveFixedJoint>true</preserveFixedJoint>
-        </gazebo>
-    </xacro:macro>
+    <!-- Sensors -->
     <xacro:macro name="gazebo_sensor_imu" params="name update_rate:=62" >
         <gazebo reference="link_sensor_imu_${name}">
@@ -106,4 +74,37 @@
         </gazebo>
     </xacro:macro>
+    <xacro:macro name="gazebo_sensor_rplidar" params="name" >
+        <gazebo reference="link_sensor_lidar_${name}">
+            <sensor name="${name}" type="gpu_lidar">
+                <update_rate>62.0</update_rate>
+                <visualize>1</visualize>
+                <always_on>true</always_on>
+                <lidar>
+                <scan>
+                    <horizontal>
+                        <samples>640</samples>
+                        <resolution>1.0</resolution>
+                        <min_angle>${-pi}</min_angle>
+                        <max_angle>${pi}</max_angle>
+                    </horizontal>
+                    <vertical>
+                        <samples>1</samples>
+                        <resolution>1</resolution>
+                        <min_angle>0</min_angle>
+                        <max_angle>0</max_angle>
+                    </vertical>
+                </scan>
+                <range>
+                    <min>0.164</min>
+                    <max>12.0</max>
+                    <resolution>0.01</resolution>
+                </range>
+                </lidar>
+            </sensor>
+        </gazebo>
+        <gazebo reference="joint_body_to_sensor_lidar_${name}">
+            <preserveFixedJoint>true</preserveFixedJoint>
+        </gazebo>
+    </xacro:macro>
     <!--
         GAZEBO
@@ -113,6 +114,6 @@
     <xacro:gazebo_reference_link_wheel name="right_rear" />
     <xacro:gazebo_reference_link_wheel name="right_front" />
+    <xacro:gazebo_sensor_imu name="imu_center" />
     <xacro:gazebo_sensor_rplidar name="rplidar_front" />
-    <xacro:gazebo_sensor_imu name="imu_center" />
     <gazebo>
         <plugin

File: urdf/macros.xacro (robot description, xacro)
@@ -170,5 +170,5 @@
         <xacro:property name="collision_x_offset" value="0.005" />
         <xacro:property name="collision_y_offset" value="0.005" />
-        <xacro:property name="collision_z_offset" value="0.005" />
+        <xacro:property name="collision_z_offset" value="${0.5 * length_z}" />
         <joint name="joint_body_to_sensor_${name}" type="fixed">
             <xacro:insert_block name="origin"/>
@@ -209,6 +209,6 @@
         <xacro:property name="length_z" value="0.06" />
         <xacro:property name="collision_x_offset" value="0" />
-        <xacro:property name="collision_y_offset" value="0.013" />
-        <xacro:property name="collision_z_offset" value="-0.019" />
+        <xacro:property name="collision_y_offset" value="0" />
+        <xacro:property name="collision_z_offset" value="${0.5 * length_z}" />
         <joint name="joint_body_to_sensor_lidar_${name}" type="fixed">
             <parent link="${parent_link}"/>

Commit message: Change the lidar shape

File: urdf/base.xacro (robot description, xacro)
@@ -211,6 +211,9 @@
     </xacro:sensor_imu>
     <!-- LIDAR -->
-    <xacro:sensor_lidar name="rplidar_front" parent_link="chassis_link">
-        <origin rpy="0 0 0" xyz="0 0 ${0.5 * chassis_height}"/>
+    <xacro:sensor_lidar
+        name="rplidar_front"
+        parent_link="chassis_link"
+        chassis_top_absolute_height="${wheel_radius + chassis_height}" />
+        <origin rpy="0 0 0" xyz="0 0 "/>
     </xacro:sensor_lidar>
     <!-- Bump -->

File: urdf/macros.xacro (robot description, xacro)
@@ -203,5 +203,5 @@
     </xacro:macro>
     <!-- Lidar sensor -->
-    <xacro:macro name="sensor_lidar" params="name parent_link *origin">
+    <xacro:macro name="sensor_lidar" params="name parent_link chassis_top_absolute_height">
         <xacro:property name="mass"     value="0.17"/>
         <xacro:property name="length_x" value="0.071" />
@@ -210,19 +210,19 @@
         <xacro:property name="collision_x_offset" value="0" />
         <xacro:property name="collision_y_offset" value="0" />
-        <xacro:property name="collision_z_offset" value="${0.5 * length_z}" />
+        <xacro:property name="collision_z_offset" value="${chassis_top_absolute_height + 0.5 * length_z}" />
         <joint name="joint_body_to_sensor_lidar_${name}" type="fixed">
             <parent link="${parent_link}"/>
             <child link="link_sensor_lidar_${name}"/>
-            <xacro:insert_block name="origin"/>
+            <origin rpy="0 0 0" xyz="${collision_x_offset} ${collision_y_offset} ${collision_z_offset}"/>
         </joint>
         <link name="link_sensor_lidar_${name}">
             <visual>
-                <origin xyz="${collision_x_offset} ${collision_y_offset} ${collision_z_offset}"/>
-                <geometry>
-                    <box size="${length_x} ${length_y} ${length_z}"/>
-                </geometry>
-            </visual>
-            <collision>
-                <origin xyz="${collision_x_offset} ${collision_y_offset} ${collision_z_offset}"/>
+                <origin rpy="0 0 0" xyz="0.0 0 0.0"/>
+                <geometry>
+                    <box size="${length_x} ${length_y} ${length_z}"/>
+                </geometry>
+            </visual>
+            <collision>
+                <origin rpy="0 0 0" xyz="0.0 0 0.0"/>
                 <geometry>
                     <box size="${length_x} ${length_y} ${length_z}"/>

Commit message: Fix incorrect XML

File: urdf/base.xacro (robot description, xacro)
@@ -215,6 +215,4 @@
         parent_link="chassis_link"
         chassis_top_absolute_height="${wheel_radius + chassis_height}" />
-        <origin rpy="0 0 0" xyz="0 0 "/>
-    </xacro:sensor_lidar>
     <!-- Bump -->
     <!-- Sonar -->

Commit message: Moving the lidar around

File: urdf/base.xacro (robot description, xacro)
@@ -214,5 +214,5 @@
         name="rplidar_front"
         parent_link="chassis_link"
-        chassis_top_absolute_height="${wheel_radius + chassis_height}" />
+        chassis_top_relative_height="${0.5 * chassis_height}" />
     <!-- Bump -->
     <!-- Sonar -->

File: urdf/macros.xacro (robot description, xacro)
@@ -203,5 +203,5 @@
     </xacro:macro>
     <!-- Lidar sensor -->
-    <xacro:macro name="sensor_lidar" params="name parent_link chassis_top_absolute_height">
+    <xacro:macro name="sensor_lidar" params="name parent_link chassis_top_relative_height">
         <xacro:property name="mass"     value="0.17"/>
         <xacro:property name="length_x" value="0.071" />
@@ -210,5 +210,5 @@
         <xacro:property name="collision_x_offset" value="0" />
         <xacro:property name="collision_y_offset" value="0" />
-        <xacro:property name="collision_z_offset" value="${chassis_top_absolute_height + 0.5 * length_z}" />
+        <xacro:property name="collision_z_offset" value="${chassis_top_relative_height}" />
         <joint name="joint_body_to_sensor_lidar_${name}" type="fixed">
             <parent link="${parent_link}"/>
@@ -218,11 +218,11 @@
         <link name="link_sensor_lidar_${name}">
             <visual>
-                <origin rpy="0 0 0" xyz="0.0 0 0.0"/>
-                <geometry>
-                    <box size="${length_x} ${length_y} ${length_z}"/>
-                </geometry>
-            </visual>
-            <collision>
-                <origin rpy="0 0 0" xyz="0.0 0 0.0"/>
+                <origin rpy="0 0 0" xyz="0.0 0 ${0.5 * length_z}"/>
+                <geometry>
+                    <box size="${length_x} ${length_y} ${length_z}"/>
+                </geometry>
+            </visual>
+            <collision>
+                <origin rpy="0 0 0" xyz="0.0 0 ${0.5 * length_z}"/>
                 <geometry>
                     <box size="${length_x} ${length_y} ${length_z}"/>
@@ -231,5 +231,5 @@
             <inertial>
                 <mass value="${mass}" />
-                <origin rpy="0 0 0" xyz="0.0 0 0.0"/>
+                <origin rpy="0 0 0" xyz="0.0 0 ${0.5 * length_z}"/>
                 <inertia
                     ixx="${(1/12) * mass * (length_y*length_y + length_z*length_z)}"
