Commit message: Set the friction coefficients for the wheels when running in Gazebo

File: urdf/gazebo.xacro (robot description, xacro)
@@ -1,4 +1,30 @@
 <?xml version="1.0" ?>
 <robot name="cratebot" xmlns:xacro="http://www.ros.org/wiki/xacro" >
+    <!--
+        GAZEBO MACROS
+    -->
+    <!--
+        Define Gazebo specific macro's here because this file isn't included if we're not running
+        Gazebo
+    -->
+    <xacro:macro name="gazebo_reference_link_wheel" params="name">
+        <gazebo reference="link_wheel_${name}">
+            <mu1>0.9</mu1>
+            <mu2>0.9</mu2>
+            <kp>500000.0</kp>
+            <kd>10.0</kd>
+            <minDepth>0.001</minDepth>
+            <maxVel>0.1</maxVel>
+            <fdir1>1 0 0</fdir1>
+            <selfCollide>true</selfCollide>
+        </gazebo>
+    </xacro:macro>
+    <!--
+        GAZEBO
+    -->
+    <xacro:gazebo_reference_link_wheel name="left_front" />
+    <xacro:gazebo_reference_link_wheel name="right_front" />
+    <xacro:gazebo_reference_link_wheel name="left_rear" />
+    <xacro:gazebo_reference_link_wheel name="right_rear" />
     <gazebo>
         <plugin filename="libign_ros2_control-system.so" name="ign_ros2_control::IgnitionROS2ControlPlugin">

Commit message: Tweaking the sensors

File: urdf/gazebo.xacro (robot description, xacro)
@@ -153,4 +153,5 @@
                 filename="libignition-gazebo-sensors-system.so"
                 name="ignition::gazebo::systems::Sensors">
+            <render_engine>ogre2</render_engine>
         </plugin>
     </gazebo>

File: urdf/macros.xacro (robot description, xacro)
@@ -171,5 +171,5 @@
         <xacro:property name="collision_y_offset" value="0.005" />
         <xacro:property name="collision_z_offset" value="${0.5 * length_z}" />
-        <joint name="joint_body_to_sensor_${name}" type="fixed">
+        <joint name="joint_body_to_sensor_imu_${name}" type="fixed">
             <xacro:insert_block name="origin"/>
             <parent link="${parent_link}"/>

Commit message: Add the update rate to the sensors

File: urdf/gazebo.xacro (robot description, xacro)
@@ -21,5 +21,5 @@
     </xacro:macro>
     <!-- Sensors -->
-    <xacro:macro name="gazebo_sensor_imu" params="name update_rate:=62" >
+    <xacro:macro name="gazebo_sensor_imu" params="name update_rate:=25" >
         <gazebo reference="link_sensor_imu_${name}">
             <sensor name="${name}" type="imu">
@@ -77,7 +77,11 @@
         <gazebo reference="link_sensor_lidar_${name}">
             <sensor name="${name}" type="gpu_lidar">
+                <!--
+                    Move the sensor up slightly from the bottom of the lidar unit.
+                -->
                 <pose>0 0 0.02 0 0 0</pose>
                 <alwaysOn>true</alwaysOn>
                 <topic>rplidar_front/scan</topic>
+                <update_rate>25</update_rate>
                 <lidarName>rplidar_front</lidarName>
                 <visualize>true</visualize>
@@ -155,4 +159,5 @@
                 name="ignition::gazebo::systems::Sensors">
             <render_engine>ogre2</render_engine>
+            <updateRate>25</updateRate>
         </plugin>
     </gazebo>
